File: _autosave-PI_Hat_TX_with_Adf4351_V1.sch (KiCad schematic (older format))
At the start: 64 parts, among them J3 RPi_GPIO, P2 4Sip200, P3 2Sip200, P4 SMA, P5 CONN_01X02, Q1 BC817-40, U1 L4940V5 1.5A

Commit message: adding dock
Parts:
- C1, C? (x18): symbol Raspberry_Pi_2m_TX_LPF_7Stage-cache:C_Small -> PI_Hat_TX_with_Adf4351_V1-rescue:C_Small-Raspberry_Pi_2m_TX_LPF_7Stage-cache
- C2, C3: symbol Raspberry_Pi_2m_TX_LPF_7Stage-cache:CP1_Small -> PI_Hat_TX_with_Adf4351_V1-rescue:CP1_Small-Raspberry_Pi_2m_TX_LPF_7Stage-cache
- D?: symbol Raspberry_Pi_2m_TX_LPF_7Stage-cache:LED -> PI_Hat_TX_with_Adf4351_V1-rescue:LED-Raspberry_Pi_2m_TX_LPF_7Stage-cache
- J3: symbol PI_Hat_TX_with_Adf4351_V1-rescue:RPi_GPIO -> PI_Hat_TX_with_Adf4351_V1-rescue:RPi_GPIO-PI_Hat_TX_with_Adf4351_V1-rescue
- J?: symbol PI_Hat_TX_with_Adf4351_V1-rescue:Conn_02x05_Odd_Even-RESCUE-PI_Hat_TX_with_Adf4351_V1 -> PI_Hat_TX_with_Adf4351_V1-rescue:Conn_02x05_Odd_Even-RESCUE-PI_Hat_TX_with_Adf4351_V1-PI_Hat_TX_with_Adf4351_V1-rescue
- L? (x8): symbol Raspberry_Pi_2m_TX_LPF_7Stage-cache:L_Small -> PI_Hat_TX_with_Adf4351_V1-rescue:L_Small-Raspberry_Pi_2m_TX_LPF_7Stage-cache
- P2: symbol Raspberry_Pi_2m_TX_LPF_7Stage-cache:Conn_01x04 -> PI_Hat_TX_with_Adf4351_V1-rescue:Conn_01x04-Raspberry_Pi_2m_TX_LPF_7Stage-cache
- P3, P5: symbol Raspberry_Pi_2m_TX_LPF_7Stage-cache:Conn_01x02 -> PI_Hat_TX_with_Adf4351_V1-rescue:Conn_01x02-Raspberry_Pi_2m_TX_LPF_7Stage-cache
- P4, P? (x2): symbol Raspberry_Pi_2m_TX_LPF_7Stage-cache:SMA -> PI_Hat_TX_with_Adf4351_V1-rescue:SMA-Raspberry_Pi_2m_TX_LPF_7Stage-cache
- Q1: symbol Raspberry_Pi_2m_TX_LPF_7Stage-cache:BC817-40 -> PI_Hat_TX_with_Adf4351_V1-rescue:BC817-40-Raspberry_Pi_2m_TX_LPF_7Stage-cache
- R1, R2, R3, R4, R5, R9, R? (x9): symbol Raspberry_Pi_2m_TX_LPF_7Stage-cache:R -> PI_Hat_TX_with_Adf4351_V1-rescue:R-Raspberry_Pi_2m_TX_LPF_7Stage-cache
- T? (x2): symbol MABA-009180-500MHz_transformer:MABA-009180-500MHz_1P_1S -> PI_Hat_TX_with_Adf4351_V1-rescue:MABA-009180-500MHz_1P_1S-MABA-009180-500MHz_transformer
- U1: symbol Raspberry_Pi_2m_TX_LPF_7Stage-cache:LM7805-RESCUE-RPi_Hat -> PI_Hat_TX_with_Adf4351_V1-rescue:LM7805-RESCUE-RPi_Hat-Raspberry_Pi_2m_TX_LPF_7Stage-cache
- U?: symbol PI_Hat_TX_with_Adf4351_V1-rescue:ADE-30 -> PI_Hat_TX_with_Adf4351_V1-rescue:ADE-30-PI_Hat_TX_with_Adf4351_V1-rescue
- U? (x4): symbol SBB2089Z-_MINI_POWER_amp_20dbm:SBB2089Z -> PI_Hat_TX_with_Adf4351_V1-rescue:SBB2089Z-SBB2089Z-_MINI_POWER_amp_20dbm
- U?: symbol PI_Hat_TX_with_Adf4351_V1-rescue:SF2124E -> PI_Hat_TX_with_Adf4351_V1-rescue:SF2124E-PI_Hat_TX_with_Adf4351_V1-rescue
- U?: symbol PI_Hat_TX_with_Adf4351_V1-rescue:SXBP-150+ -> PI_Hat_TX_with_Adf4351_V1-rescue:SXBP-150+-PI_Hat_TX_with_Adf4351_V1-rescue
